Commit message: Updated URDF file.

File: src/ros_rover/urdf/viam_rover.urdf (robot description, URDF)
Before this commit: robot viam_rover, 5 links, 4 joints
Joints:
- joint base_link_to_chassis: origin xyz=0 0 0 -> xyz=0 0 0.015
- joint laser_joint: origin xyz=0.05 0 0.09 rpy=0 0 0 -> xyz=0.05 0 0.07 rpy=0 0 0

Commit message: Updated URDF file.

File: src/ros_rover/urdf/viam_rover.urdf (robot description, URDF)
Before this commit: robot viam_rover, 5 links, 4 joints
Links:
- added link caster_wheel; visual sphere radius=0.015
Joints:
- added joint caster_joint: type fixed, parent chassis, child caster_wheel, origin xyz=0.08 0 0 rpy=0 0 0
- joint left_wheel_joint: origin xyz=0 0.08 0.0325 rpy=-1.5708 0 0 -> xyz=0 0.10 0.0325 rpy=-1.5708 0 0
- joint right_wheel_joint: origin xyz=0 -0.08 0.0325 rpy=1.5708 0 0 -> xyz=0 -0.10 0.0325 rpy=1.5708 0 0

Commit message: Updated URDF file.

File: src/ros_rover/urdf/viam_rover.urdf (robot description, URDF)
Before this commit: robot viam_rover, 6 links, 5 joints
Joints:
- joint caster_joint: origin xyz=0.08 0 0 rpy=0 0 0 -> xyz=-0.08 0 0 rpy=0 0 0
- joint laser_joint: origin xyz=0.05 0 0.07 rpy=0 0 0 -> xyz=-0.02 0 0.07 rpy=0 0 0
- joint left_wheel_joint: origin xyz=0 0.10 0.0325 rpy=-1.5708 0 0 -> xyz=0.08 0.10 0.0325 rpy=-1.5708 0 0
- joint right_wheel_joint: origin xyz=0 -0.10 0.0325 rpy=1.5708 0 0 -> xyz=0.08 -0.10 0.0325 rpy=1.5708 0 0

Commit message: Updated URDF file.

File: src/ros_rover/urdf/viam_rover.urdf (robot description, URDF)
Before this commit: robot viam_rover, 6 links, 5 joints
Links:
- link chassis: geometry visual box size=0.31 0.21 0.07
Joints:
- joint base_link_to_chassis: origin xyz=0 0 0.015 -> xyz=-0.08 0 0.02
- joint caster_joint: origin xyz=-0.08 0 0 rpy=0 0 0 -> xyz=-0.14 0 0 rpy=0 0 0
- joint laser_joint: origin xyz=-0.02 0 0.07 rpy=0 0 0 -> xyz=0.05 0 0.07 rpy=0 0 0
- joint left_wheel_joint: axis 0 0 1 -> 0 1 0; origin xyz=0.08 0.10 0.0325 rpy=-1.5708 0 0 -> xyz=0 0.12 0.0125 rpy=0 0 0
- joint right_wheel_joint: axis 0 0 1 -> 0 1 0; origin xyz=0.08 -0.10 0.0325 rpy=1.5708 0 0 -> xyz=0 -0.12 0.0125 rpy=0 0 0

Commit message: Updated URDF file.

File: src/ros_rover/urdf/viam_rover.urdf (robot description, URDF)
Before this commit: robot viam_rover, 6 links, 5 joints
Joints:
- joint base_link_to_chassis: origin xyz=-0.08 0 0.02 -> xyz=-0.08 0 0.015
- joint left_wheel_joint: origin xyz=0 0.12 0.0125 rpy=0 0 0 -> xyz=0 0.12 0.0325 rpy=0 0 0
- joint right_wheel_joint: origin xyz=0 -0.12 0.0125 rpy=0 0 0 -> xyz=0 -0.12 0.0325 rpy=0 0 0

Commit message: Updated URDF file.

File: src/ros_rover/urdf/viam_rover.urdf (robot description, URDF)
Before this commit: robot viam_rover, 6 links, 5 joints
Joints:
- joint base_link_to_chassis: origin xyz=-0.08 0 0.015 -> xyz=0 0 0.015
- joint caster_joint: origin xyz=-0.14 0 0 rpy=0 0 0 -> xyz=-0.12 0 0 rpy=0 0 0
- joint laser_joint: origin xyz=0.05 0 0.07 rpy=0 0 0 -> xyz=0.08 0 0.07 rpy=0 0 0
- joint left_wheel_joint: origin xyz=0 0.12 0.0325 rpy=0 0 0 -> xyz=0.10 0.13 0.0325 rpy=0 0 0
- joint right_wheel_joint: origin xyz=0 -0.12 0.0325 rpy=0 0 0 -> xyz=0.10 -0.13 0.0325 rpy=0 0 0

Commit message: Updated URDF file.

File: src/ros_rover/urdf/viam_rover.urdf (robot description, URDF)
Before this commit: robot viam_rover, 6 links, 5 joints
Links:
- removed link caster_wheel
- removed link left_wheel
- removed link right_wheel
- added link front_left_wheel; visual cylinder length=0.025 radius=0.0325
- added link front_right_wheel; visual cylinder length=0.025 radius=0.0325
- added link rear_caster; visual sphere radius=0.015
Joints:
- removed joint caster_joint
- removed joint left_wheel_joint
- removed joint right_wheel_joint
- added joint front_left_wheel_joint: type continuous, parent base_link, child front_left_wheel, origin xyz=0.12 0.13 0.0325 rpy=0 0 0, axis 0 1 0
- added joint front_right_wheel_joint: type continuous, parent base_link, child front_right_wheel, origin xyz=0.12 -0.13 0.0325 rpy=0 0 0, axis 0 1 0
- added joint rear_caster_joint: type fixed, parent base_link, child rear_caster, origin xyz=-0.12 0 0.015 rpy=0 0 0
- joint base_link_to_chassis: origin xyz=0 0 0.015 -> xyz=0 0 0.05
- joint laser_joint: origin xyz=0.08 0 0.07 rpy=0 0 0 -> xyz=0.08 0 0.035 rpy=0 0 0
