Commit message: Fix URDF/driver joint name mismatch and update physical constants
- Fix wheel display bug: rename URDF joints to left/right_wheel_joint to
  match JointState names published by viam_driver.py
- Correct wheel geometry: radius 35mm (was 32.5mm), separation 230mm
  (was 160mm), Y offsets ±115mm to reflect wheels protruding through chassis
- Replace rover_bringup static laser TF (conflicted with URDF) with RSP include
- Add display.launch.py for RVIZ preview without hardware
- Add imu_link placeholder for upcoming ICM20948 integration
- Fix encoder callbacks to decrement ticks when driving in reverse

Co-Authored-By: Claude Sonnet 4.6 <noreply@anthropic.com>

File: src/ros_rover/urdf/viam_rover.urdf (robot description, URDF)
Before this commit: robot viam_rover, 6 links, 5 joints
Links:
- removed link front_left_wheel
- removed link front_right_wheel
- added link imu_link; visual box size=0.02 0.02 0.004
- added link left_wheel; visual cylinder length=0.025 radius=0.035
- added link right_wheel; visual cylinder length=0.025 radius=0.035
Joints:
- removed joint front_left_wheel_joint
- removed joint front_right_wheel_joint
- added joint imu_joint: type fixed, parent chassis, child imu_link, origin xyz=0 0 0.035 rpy=0 0 0
- added joint left_wheel_joint: type continuous, parent base_link, child left_wheel, origin xyz=0.12 0.115 0.035 rpy=0 0 0, axis 0 1 0
- added joint right_wheel_joint: type continuous, parent base_link, child right_wheel, origin xyz=0.12 -0.115 0.035 rpy=0 0 0, axis 0 1 0
- joint base_link_to_chassis: origin xyz=0 0 0.05 -> xyz=0 0 0.05 rpy=0 0 0
